File: hardware/hardware.sch (KiCad schematic (older format))
At the start: 52 parts, among them IC1 TP4056, J1 eink, J2 TC2030-IDV-NL, J3 Vin, Q1 AO3401A, Q2 AO3400A, U1 STM32L031F6Px, U2 XC6206P332MR-G, U3 CAT24C256

Commit message: Add J1 connector
Parts:
- J1: footprint (none) -> Dianwei:FPC_24
Changed lines of the file:
@@
 F 0 "J1" H 8842 3085 50  0000 C CNN
 F 1 "eink" H 8842 2994 50  0000 C CNN
-F 2 "" H 8950 1800 50  0001 C CNN
+F 2 "Dianwei:FPC_24" H 8950 1800 50  0001 C CNN
 F 3 "../documentation/24 Pins 0.5mm Pitch ZIF Connector Drawing.pdf" H 8950 1800 50  0001 C CNN
 	1    8950 1800

Commit message: Placed components
Parts:
- L1: value 10uA -> 10 uH; LCSC C86073 -> C86069
Connections:
- wire segments 158 -> 159
Other:
- moved on the sheet: D1, D2, R1, R2
Changed lines of the file:
@@
 P 4300 1250
 F 0 "L1" V 4490 1250 50  0000 C CNN
-F 1 "10uA" V 4399 1250 50  0000 C CNN
+F 1 "10 uH" V 4399 1250 50  0000 C CNN
 F 2 "Inductor_SMD:L_1210_3225Metric" H 4300 1250 50  0001 C CNN
-F 3 "https://datasheet.lcsc.com/szlcsc/Murata-Electronics-LQH32PN100MNCL_C86073.pdf" H 4300 1250 50  0001 C CNN
-F 4 "C86073" V 4300 1250 50  0001 C CNN "LCSC"
+F 3 "https://datasheet.lcsc.com/szlcsc/Murata-Electronics-LQH32CN100K33L_C86069.pdf" H 4300 1250 50  0001 C CNN
+F 4 "C86069" V 4300 1250 50  0001 C CNN "LCSC"
 	1    4300 1250
 	0    -1   -1   0
@@
 L Device:LED_Small D2
 U 1 1 5DEC3843
-P 1300 3800
-F 0 "D2" V 1300 3700 50  0000 R CNN
-F 1 "RED" V 1200 3750 50  0000 R CNN
-F 2 "Diode_SMD:D_0603_1608Metric" V 1300 3800 50  0001 C CNN
-F 3 "https://datasheet.lcsc.com/szlcsc/Hubei-KENTO-Elec-KT-0603R_C2286.pdf" V 1300 3800 50  0001 C CNN
-F 4 "C2286" V 1300 3800 50  0001 C CNN "LCSC"
-	1    1300 3800
-	0    -1   -1   0
+P 1600 4000
+F 0 "D2" H 1550 3950 50  0000 R CNN
+F 1 "RED" H 1550 4050 50  0000 R CNN
+F 2 "Diode_SMD:D_0603_1608Metric" V 1600 4000 50  0001 C CNN
+F 3 "https://datasheet.lcsc.com/szlcsc/Hubei-KENTO-Elec-KT-0603R_C2286.pdf" V 1600 4000 50  0001 C CNN
+F 4 "C2286" V 1600 4000 50  0001 C CNN "LCSC"
+	1    1600 4000
+	-1   0    0    1
 $EndComp
 $Comp
 L Device:R_Small R2
 U 1 1 5DEC54FA
-P 1700 4000
-F 0 "R2" V 1650 3800 50  0000 C CNN
-F 1 "2k" V 1750 3800 50  0000 C CNN
-F 2 "Resistor_SMD:R_0402_1005Metric" H 1700 4000 50  0001 C CNN
-F 3 "https://datasheet.lcsc.com/szlcsc/Uniroyal-Elec-0402WGF2001TCE_C4109.pdf" H 1700 4000 50  0001 C CNN
-F 4 "C4109" V 1700 4000 50  0001 C CNN "LCSC"
-	1    1700 4000
-	0    1    1    0
-$EndComp
-Wire Wire Line
-	1000 3700 1300 3700
+P 1400 3800
+F 0 "R2" H 1300 3850 50  0000 C CNN
+F 1 "2k" H 1300 3750 50  0000 C CNN
+F 2 "Resistor_SMD:R_0402_1005Metric" H 1400 3800 50  0001 C CNN
+F 3 "https://datasheet.lcsc.com/szlcsc/Uniroyal-Elec-0402WGF2001TCE_C4109.pdf" H 1400 3800 50  0001 C CNN
+F 4 "C4109" V 1400 3800 50  0001 C CNN "LCSC"
+	1    1400 3800
+	-1   0    0    1
+$EndComp
 $Comp
 L Device:LED_Small D1
 U 1 1 5DECE3AB
-P 1000 4000
-F 0 "D1" V 1046 3932 50  0000 R CNN
-F 1 "GREEN" V 955 3932 50  0000 R CNN
-F 2 "Diode_SMD:D_0603_1608Metric" V 1000 4000 50  0001 C CNN
-F 3 "https://datasheet.lcsc.com/szlcsc/Everlight-Elec-19-217-GHC-YR1S2-3T_C72043.pdf" V 1000 4000 50  0001 C CNN
-F 4 "C72043" V 1000 4000 50  0001 C CNN "LCSC"
-	1    1000 4000
-	0    -1   -1   0
-$EndComp
-Connection ~ 1300 3700
-Wire Wire Line
-	1300 3700 1800 3700
-Wire Wire Line
-	1600 4000 1300 4000
-Wire Wire Line
-	1300 4000 1300 3900
+P 1450 4200
+F 0 "D1" H 1400 4150 50  0000 R CNN
+F 1 "GREEN" H 1400 4250 50  0000 R CNN
+F 2 "Diode_SMD:D_0603_1608Metric" V 1450 4200 50  0001 C CNN
+F 3 "https://datasheet.lcsc.com/szlcsc/Everlight-Elec-19-217-GHC-YR1S2-3T_C72043.pdf" V 1450 4200 50  0001 C CNN
+F 4 "C72043" V 1450 4200 50  0001 C CNN "LCSC"
+	1    1450 4200
+	-1   0    0    1
+$EndComp
 Wire Wire Line
 	1000 3900 1000 3700
@@
 L Device:R_Small R1
 U 1 1 5DED5C57
-P 1450 4200
-F 0 "R1" V 1400 4000 50  0000 C CNN
-F 1 "2k" V 1500 4000 50  0000 C CNN
-F 2 "Resistor_SMD:R_0402_1005Metric" H 1450 4200 50  0001 C CNN
-F 3 "https://datasheet.lcsc.com/szlcsc/Uniroyal-Elec-0402WGF2001TCE_C4109.pdf" H 1450 4200 50  0001 C CNN
-F 4 "C4109" V 1450 4200 50  0001 C CNN "LCSC"
-	1    1450 4200
-	0    1    1    0
+P 1000 4000
+F 0 "R1" H 900 4050 50  0000 C CNN
+F 1 "2k" H 900 3950 50  0000 C CNN
+F 2 "Resistor_SMD:R_0402_1005Metric" H 1000 4000 50  0001 C CNN
+F 3 "https://datasheet.lcsc.com/szlcsc/Uniroyal-Elec-0402WGF2001TCE_C4109.pdf" H 1000 4000 50  0001 C CNN
+F 4 "C4109" V 1000 4000 50  0001 C CNN "LCSC"
+	1    1000 4000
+	-1   0    0    1
 $EndComp
 Wire Wire Line
@@
 	2750 2150 3450 2150
 Text Label 2850 2150 0    50   ~ 0
-EINK_CS
+EINK_BUSY
 Wire Wire Line
 	2750 2450 3450 2450
@@
 	2750 1750 3450 1750
 Text Label 2850 1550 0    50   ~ 0
-EINK_BUSY
+EINK_CS
 Wire Wire Line
 	5800 4000 5800 3700
@@
 	1    0    0    -1
 $EndComp
+Wire Wire Line
+	1000 3700 1400 3700
+Connection ~ 1400 3700
+Wire Wire Line
+	1400 3700 1800 3700
+Wire Wire Line
+	1800 4000 1700 4000
+Wire Wire Line
+	1500 4000 1400 4000
+Wire Wire Line
+	1400 4000 1400 3900
 $EndSCHEMATC

Commit message: Update voltage divider
Parts:
- removed TP1: TP_VBAT, TestPoint:TestPoint_Pad_D1.5mm, symbol Connector:TestPoint_Alt
- R10: value 422k -> 39k; LCSC C60390 -> C25783
- R9: value 150k -> 15k; LCSC C25755 -> C25756
Connections:
- net labels added: VBAT_ON
- wire segments 159 -> 160
- no-connect marks 5 -> 4
Changed lines of the file:
@@
 P 1600 5500
 F 0 "R9" V 1404 5500 50  0000 C CNN
-F 1 "150k" V 1495 5500 50  0000 C CNN
+F 1 "15k" V 1495 5500 50  0000 C CNN
 F 2 "Resistor_SMD:R_0402_1005Metric" H 1600 5500 50  0001 C CNN
-F 3 "https://datasheet.lcsc.com/szlcsc/Uniroyal-Elec-0402WGF1503TCE_C25755.pdf" H 1600 5500 50  0001 C CNN
-F 4 "C25755" V 1600 5500 50  0001 C CNN "LCSC"
+F 3 "" H 1600 5500 50  0001 C CNN
+F 4 "C25756" V 1600 5500 50  0001 C CNN "LCSC"
 	1    1600 5500
 	0    1    1    0
@@
 P 1950 5650
 F 0 "R10" H 2009 5696 50  0000 L CNN
-F 1 "422k" H 2009 5605 50  0000 L CNN
+F 1 "39k" H 2009 5605 50  0000 L CNN
 F 2 "Resistor_SMD:R_0402_1005Metric" H 1950 5650 50  0001 C CNN
-F 3 "https://datasheet.lcsc.com/szlcsc/Uniroyal-Elec-0402WGF4223TCE_C60390.pdf" H 1950 5650 50  0001 C CNN
-F 4 "C60390" H 1950 5650 50  0001 C CNN "LCSC"
+F 3 "" H 1950 5650 50  0001 C CNN
+F 4 "C25783" H 1950 5650 50  0001 C CNN "LCSC"
 	1    1950 5650
 	1    0    0    -1
@@
 Wire Wire Line
 	1950 5500 1950 5550
-Wire Wire Line
-	1950 5500 2450 5500
-Connection ~ 1950 5500
-Text Label 2200 5500 0    50   ~ 0
-VBAT
 $Comp
 L Memory_EEPROM:CAT24C256 U3
@@
 Text Label 7600 5200 0    50   ~ 0
 TX
-Connection ~ 800  5850
-Wire Wire Line
-	800  5850 1950 5850
 Wire Wire Line
 	1950 5750 1950 5850
@@
 	1550 900  1900 900
 NoConn ~ 1750 2350
-NoConn ~ 1750 2450
 $Comp
 L Connector:Conn_01x02_Male J3
@@
 	8300 3700 8050 3700
 Connection ~ 8050 3700
-$Comp
-L Connector:TestPoint_Alt TP1
-U 1 1 5E03CE53
-P 2450 5500
-F 0 "TP1" H 2508 5618 50  0000 L CNN
-F 1 "TP_VBAT" H 2508 5527 50  0000 L CNN
-F 2 "TestPoint:TestPoint_Pad_D1.5mm" H 2650 5500 50  0001 C CNN
-F 3 "~" H 2650 5500 50  0001 C CNN
-	1    2450 5500
-	1    0    0    -1
-$EndComp
 Wire Wire Line
 	1000 3700 1400 3700
@@
 Wire Wire Line
 	1400 4000 1400 3900
+Connection ~ 1950 5500
+Wire Wire Line
+	1950 5500 2450 5500
+Text Label 2200 5500 0    50   ~ 0
+VBAT
+Wire Wire Line
+	1750 2450 1200 2450
+Text Label 1250 2450 0    50   ~ 0
+VBAT_ON
+Wire Wire Line
+	1950 5850 2450 5850
+Text Label 2050 5850 0    50   ~ 0
+VBAT_ON
 $EndSCHEMATC
