File: hardware/hardware.kicad_pcb (KiCad board)
At the start: 4 copper layers, 39.4 x 38.1 mm, 52 parts, among them IC1 TP4056, J1 eink, J2 TC2030-IDV-NL, J3 Vin, Q1 AO3401A, Q2 AO3400A, U1 STM32L031F6Px, U2 XC6206P332MR-G, U3 CAT24C256

Commit message: Board routed
Parts:
- removed TP1: TP_VBAT, TestPoint:TestPoint_Pad_D1.5mm
- R10: value 422k -> 39k
- R9: value 150k -> 15k
- moved C2 3.85 mm to (38.0, 120.1)
- moved R9 3.80 mm to (39.9, 137.5)
- moved R10 3.42 mm to (39.9, 139.1)
- turned C11 to 180 degrees
Connections:
- R10 pad 2: GND -> /VBAT_ON
- U1 pad 3: Net-(U1-Pad3) -> /VBAT_ON
Routing:
- net +3V3: track 4.19 -> 33.0 mm, vias 1 -> 10
- net /EINK_RESET: track 0.00 -> 26.7 mm, vias 0 -> 1
- net /EINK_CS: track 0.00 -> 26.5 mm, vias 0 -> 1
- net /EINK_DC: track 0.00 -> 25.2 mm, vias 0 -> 1
- net /SPI_SDI: track 0.00 -> 23.1 mm, vias 0 -> 1
- net /EINK_BUSY: track 0.00 -> 21.7 mm, vias 0 -> 1
- net /SPI_SCK: track 0.00 -> 19.8 mm, vias 0 -> 1
- net /RX: track 0.00 -> 19.5 mm, vias 0 -> 1
- net +BATT: track 7.76 -> 24.1 mm, vias 1 -> 3
- net Net-(C4-Pad1): track 0.00 -> 13.9 mm
- net Net-(C4-Pad2): track 0.00 -> 12.4 mm
- net /VBAT_ON: track 0.00 -> 12.2 mm, vias 0 -> 2
- net /I2C_SDA: track 0.00 -> 11.2 mm
- net /SWCLK: track 0.00 -> 11.1 mm, vias 0 -> 1
- net /RESE: track 0.00 -> 10.9 mm, vias 0 -> 1
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- added copper zone on B.Cu, net GND
- added copper zone on F.Cu, net GND
Other:
- board size 39.4 x 38.1 mm -> 41.4 x 38.1 mm
- board text added: "G T 3"
- board text added: "JLCJLCJLCJLC"
- board text added: "Photokey v1.0"
- board text added: "R C I"
- board text added: "ioPush.net"
